File: PCB/PCB.kicad_pcb (KiCad board)
At the start: 2 copper layers, 99.9 x 99.9 mm, 64 parts, among them J1 MCU POWER, J10 Conn_01x03, J11 Conn_01x03, J12 Conn_01x03, J13 Conn_01x03, J14 Conn_01x03, J15 Conn_01x03, J16 Conn_01x03, J17 Conn_01x03, J18 Conn_01x03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

Commit message: Update code folder
Parts:
- removed R7, R8: 6.8k, Resistor_THT:R_Axial_DIN0207_L6.3mm_D2.5mm_P7.62mm_Horizontal
- CFF1, CFF2, CFF3: value 100nF -> 33nF
- COUT1, COUT2, COUT3: value 220uF/50V -> 330uF/25V
- renumbered U3 to U2, U2 to U3
Connections:
- J10 pad 1: PMW_8 -> PMW8_2
- J11 pad 1: PMW_9 -> PMW7_2
- J12 pad 1: PMW_10 -> PMW15_1
- J13 pad 1: PMW_11 -> PMW14_1
- J14 pad 1: PMW_12 -> PMW13_1
- J15 pad 1: PMW_13 -> PMW12_1
- J16 pad 1: PMW_14 -> PMW11_1
- J17 pad 1: PMW_15 -> PMW10_1
- J18 pad 1: PMW_16 -> PMW9_1
- J19 pad 1: PMW_17 -> PMW8_1
- J20 pad 1: PMW_18 -> PMW7_1
- J3 pad 1: PMW_1 -> PMW15_2
- J4 pad 1: PMW_2 -> PMW14_2
- J5 pad 1: PMW_3 -> PMW13_2
- J6 pad 1: PMW_4 -> PMW12_2
- J7 pad 1: PMW_5 -> PMW11_2
- J8 pad 1: PMW_6 -> PMW10_2
- J9 pad 1: PMW_7 -> PMW9_2
- U2 pad 1: PMW_10 -> unconnected-(U2-PWM0-Pad1)
- U2 pad 10: unconnected-(U3-PWM10-Pad10) -> PMW9_1
- U2 pad 11: unconnected-(U3-PWM11-Pad11) -> PMW10_1
- U2 pad 12: unconnected-(U3-PWM12-Pad12) -> PMW11_1
- U2 pad 13: unconnected-(U3-PMW13-Pad13) -> PMW12_1
- U2 pad 14: unconnected-(U3-PMW14-Pad14) -> PMW13_1
- U2 pad 15: unconnected-(U3-PMW15-Pad15) -> PMW14_1
- U2 pad 16: unconnected-(U3-PMW16-Pad16) -> PMW15_1
- U2 pad 2: PMW_11 -> unconnected-(U2-PWM1-Pad2)
- U2 pad 3: PMW_12 -> unconnected-(U2-PWM2-Pad3)
- U2 pad 4: PMW_13 -> unconnected-(U2-PWM3-Pad4)
- U2 pad 5: PMW_14 -> unconnected-(U2-PWM4-Pad5)
- U2 pad 6: PMW_15 -> unconnected-(U2-PWM5-Pad6)
- U2 pad 7: PMW_16 -> unconnected-(U2-PWM6-Pad7)
- U2 pad 8: PMW_17 -> PMW7_1
- U2 pad 9: PMW_18 -> PMW8_1
- U3 pad 1: PMW_1 -> unconnected-(U3-PWM0-Pad1)
- U3 pad 10: unconnected-(U2-PWM10-Pad10) -> PMW9_2
- U3 pad 11: unconnected-(U2-PWM11-Pad11) -> PMW10_2
- U3 pad 12: unconnected-(U2-PWM12-Pad12) -> PMW11_2
- U3 pad 13: unconnected-(U2-PMW13-Pad13) -> PMW12_2
- U3 pad 14: unconnected-(U2-PMW14-Pad14) -> PMW13_2
- U3 pad 15: unconnected-(U2-PMW15-Pad15) -> PMW14_2
- U3 pad 16: unconnected-(U2-PMW16-Pad16) -> PMW15_2
- U3 pad 2: PMW_2 -> unconnected-(U3-PWM1-Pad2)
- U3 pad 3: PMW_3 -> unconnected-(U3-PWM2-Pad3)
- U3 pad 4: PMW_4 -> unconnected-(U3-PWM3-Pad4)
- U3 pad 5: PMW_5 -> unconnected-(U3-PWM4-Pad5)
- U3 pad 6: PMW_6 -> unconnected-(U3-PWM5-Pad6)
- U3 pad 7: PMW_7 -> unconnected-(U3-PWM6-Pad7)
- U3 pad 8: PMW_8 -> PMW7_2
- U3 pad 9: PMW_9 -> PMW8_2
Routing:
- net PMW_8: track 51.5 -> 0.00 mm, vias 2 -> 0
- net PMW8_2: track 0.00 -> 51.5 mm, vias 0 -> 2
- net PMW_7: track 43.4 -> 0.00 mm
- net PMW9_2: track 0.00 -> 43.4 mm
- net 5V_MCU: track 195.0 -> 153.6 mm
- net PMW_6: track 40.3 -> 0.00 mm, vias 2 -> 0
- net PMW10_2: track 0.00 -> 40.3 mm, vias 0 -> 2
- net PMW_9: track 40.3 -> 0.00 mm
- net PMW7_2: track 0.00 -> 40.3 mm
- net PMW_4: track 36.1 -> 0.00 mm, vias 2 -> 0
- net PMW12_2: track 0.00 -> 36.1 mm, vias 0 -> 2
- net PMW_17: track 34.6 -> 0.00 mm
- net PMW8_1: track 0.00 -> 34.6 mm
- net PMW_11: track 33.5 -> 0.00 mm, vias 2 -> 0
- net PMW14_1: track 0.00 -> 33.5 mm, vias 0 -> 2
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