File: PCB/PCB.kicad_sch (KiCad schematic)
At the start: 64 parts, among them J1 MCU POWER, J10 Conn_01x03, J11 Conn_01x03, J12 Conn_01x03, J13 Conn_01x03, J14 Conn_01x03, J15 Conn_01x03, J16 Conn_01x03, J17 Conn_01x03, J18 Conn_01x03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

Commit message: Update code folder
Parts:
- removed R7, R8: 6.8k, Resistor_THT:R_Axial_DIN0207_L6.3mm_D2.5mm_P7.62mm_Horizontal, symbol Device:R
- CFF1, CFF2, CFF3: value 100nF -> 33nF
- COUT1, COUT2, COUT3: value 220uF/50V -> 330uF/25V
- renumbered U3 to U2, U2 to U3
Connections:
- net PMW9_2: now reaches U3.10 (PWM9)
- net PMW9_2: now also J9.1 (Pin_1)
- net PMW10_2: now reaches U3.11 (PWM10)
- net PMW10_2: now also J8.1 (Pin_1)
- net PMW11_2: now reaches U3.12 (PWM11)
- net PMW11_2: now also J7.1 (Pin_1)
- net PMW12_2: now reaches U3.13 (PMW12)
- net PMW12_2: now also J6.1 (Pin_1)
- net PMW13_2: now reaches U3.14 (PMW13)
- net PMW13_2: now also J5.1 (Pin_1)
- net PMW14_2: now reaches U3.15 (PMW14)
- net PMW14_2: now also J4.1 (Pin_1)
- net PMW15_2: now reaches U3.16 (PMW15)
- net PMW15_2: now also J3.1 (Pin_1)
- net PMW9_1: now reaches U2.10 (PWM9)
- net PMW9_1: now also J18.1 (Pin_1)
- net PMW10_1: now reaches U2.11 (PWM10)
- net PMW10_1: now also J17.1 (Pin_1)
- net PMW11_1: now reaches U2.12 (PWM11)
- net PMW11_1: now also J16.1 (Pin_1)
- net PMW12_1: now reaches U2.13 (PMW12)
- net PMW12_1: now also J15.1 (Pin_1)
- net PMW13_1: now reaches U2.14 (PMW13)
- net PMW13_1: now also J14.1 (Pin_1)
- net PMW14_1: now reaches U2.15 (PMW14)
- net PMW14_1: now also J13.1 (Pin_1)
- net PMW15_1: now reaches U2.16 (PMW15)
- net PMW15_1: now also J12.1 (Pin_1)
- net PMW_1: no longer names the net of U3.1 (PWM0)
- net PMW_1: no longer J3.1 (Pin_1)
- net PMW_10: no longer names the net of U2.1 (PWM0)
- net PMW_10: no longer J12.1 (Pin_1)
- net PMW_11: no longer names the net of U2.2 (PWM1)
- net PMW_11: no longer J13.1 (Pin_1)
- net PMW_12: no longer names the net of U2.3 (PWM2)
- net PMW_12: no longer J14.1 (Pin_1)
- net PMW_13: no longer names the net of U2.4 (PWM3)
- net PMW_13: no longer J15.1 (Pin_1)
- net PMW_14: no longer names the net of U2.5 (PWM4)
- net PMW_14: no longer J16.1 (Pin_1)
- net PMW_15: no longer names the net of U2.6 (PWM5)
- net PMW_15: no longer J17.1 (Pin_1)
- net PMW_16: no longer names the net of U2.7 (PWM6)
- net PMW_16: no longer J18.1 (Pin_1)
- net PMW_17 renamed PMW7_1
- net PMW7_1: now also J20.1 (Pin_1); no longer J19.1 (Pin_1)
- net PMW_18 renamed PMW8_1
- net PMW8_1: now also J19.1 (Pin_1); no longer J20.1 (Pin_1)
- net PMW_2: no longer names the net of U3.2 (PWM1)
- net PMW_2: no longer J4.1 (Pin_1)
- net PMW_3: no longer names the net of U3.3 (PWM2)
- net PMW_3: no longer J5.1 (Pin_1)
- net PMW_4: no longer names the net of U3.4 (PWM3)
- net PMW_4: no longer J6.1 (Pin_1)
- net PMW_5: no longer names the net of U3.5 (PWM4)
- net PMW_5: no longer J7.1 (Pin_1)
- net PMW_6: no longer names the net of U3.6 (PWM5)
- net PMW_6: no longer J8.1 (Pin_1)
- net PMW_7: no longer names the net of U3.7 (PWM6)
- net PMW_7: no longer J9.1 (Pin_1)
- net PMW_8 renamed PMW7_2
- net PMW7_2: now also J11.1 (Pin_1); no longer J10.1 (Pin_1)
- net PMW_9 renamed PMW8_2
- net PMW8_2: now also J10.1 (Pin_1); no longer J11.1 (Pin_1)
- no-connect marks 53 -> 52
Other:
- moved on the sheet: J10
